File: PixiFlood_PTH.brd (EAGLE design)
At the start: 43 x 46 mm, 37 parts, among them IC1 WS2811-SOP8, IC2 78L05Z, T1 2N3904, T2 2N3904, T3 2N3904, U1 PT4115B89E, U2 PT4115B89E, U3 PT4115B89E, X1 22-23-2031, X2 22-23-2031

Commit message: Version 9 of the Driver
Parts:
- R1, R2, R3: value .33R -> .3R
- U1, U2, U3: value PT4115B89E -> PT4115B89E-A2; device drivers:SOT89-5 -> drivers:SOT89-5-A
- moved TP1 33.0 mm to (15.2, 5.08)
- moved TP4 11.7 mm to (40.6, 2.54)
- moved TP5 11.4 mm to (40.6, 10.2)
- moved TP3 9.83 mm to (40.6, 19.1)
- moved C2 8.27 mm to (23.5, 36.4), turned to 220 degrees
- moved TP7 5.08 mm to (36.8, 10.2)
- moved TP8 4.62 mm to (36.8, 2.54)
- moved T3 4.06 mm to (38.1, 6.35)
- moved IC2 3.61 mm to (29.5, 37.3), turned to 180 degrees
- moved TP6 3.24 mm to (36.8, 19.1)
- moved TP2 3.14 mm to (33.7, 35.4)
- moved R4 3.05 mm to (41.9, 30.6), flipped to the bottom
- moved T2 2.68 mm to (38.1, 15.2)
- moved R5 1.65 mm to (41.9, 19.4), flipped to the bottom
- moved L1 1.09 mm to (30.9, 24.3)
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Connections:
- net GND: now also U1.2@1, U1.2@2, U1.2@3, U2.2@1, U2.2@2, U2.2@3, U3.2@1, U3.2@2, U3.2@3; no longer U1.2A, U1.2A@1, U1.2A@2, U1.2A@3, U1.2A@4, U2.2A, U2.2A@1, U2.2A@2, U2.2A@3, U2.2A@4, U3.2A, U3.2A@1, U3.2A@2, U3.2A@3, U3.2A@4
Routing:
- net N$18: track 25.2 -> 31.4 mm, vias 2 -> 1
- net +12V: track 98.1 -> 102.3 mm
- net GREEN: track 14.1 -> 18.1 mm
- net N$20: track 12.3 -> 15.5 mm
- net +5V: track 42.1 -> 45.2 mm
- net RED: track 14.3 -> 17.2 mm
- net BLUE: track 14.8 -> 17.7 mm
- net N$15: track 44.8 -> 42.2 mm, vias 2 -> 1
- net ROUT: track 41.1 -> 42.3 mm
- net N$2: track 9.14 -> 9.68 mm
- net N$10: track 40.3 -> 39.8 mm
- net N$1: track 8.94 -> 8.43 mm
Other:
- board text added: "V1.9"
- board text removed: "V1.7"
