File: PixiFlood_PTH.brd (EAGLE design)
At the start: 43 x 46 mm, 37 parts, among them IC1 WS2811-SOP8, IC2 78L05Z, T1 2N3904, T2 2N3904, T3 2N3904, U1 PT4115B89E-A2, U2 PT4115B89E-A2, U3 PT4115B89E-A2, X1 22-23-2031, X2 22-23-2031

Commit message: added 20w board
Parts:
- U1, U2, U3: value PT4115B89E-A2 -> PT4115B89E; device drivers:SOT89-5-A -> drivers:SOT89-5
- moved TP3 1.27 mm to (39.4, 19.1)
- moved TP5 1.27 mm to (39.4, 10.2)
- moved TP6 1.27 mm to (36.8, 19.1)
- moved TP7 1.27 mm to (36.8, 10.2)
- moved TP4 1.27 mm to (39.2, 2.16)
- moved TP8 1.27 mm to (36.3, 2.16)
Routing:
- net N$20: track 16.0 -> 15.0 mm
- net N$18: track 31.4 -> 30.7 mm
- net RED: track 17.4 -> 16.8 mm
Changed lines of the file:
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@@
 </autorouter>
 <elements>
-<element name="U1" library="drivers" package="SOT89-5-A" value="PT4115B89E-A2" x="24.637715625" y="24.4330375" smashed="yes" rot="R90">
+<element name="U1" library="drivers" package="SOT89-5" value="PT4115B89E" x="24.637715625" y="24.4330375" smashed="yes" rot="R90">
 <attribute name="NAME" x="25.209215625" y="22.9090375" size="0.6096" layer="25" rot="R180"/>
 </element>
-<element name="U2" library="drivers" package="SOT89-5-A" value="PT4115B89E-A2" x="24.13450625" y="16.641321875" smashed="yes" rot="R90">
+<element name="U2" library="drivers" package="SOT89-5" value="PT4115B89E" x="24.13450625" y="16.641321875" smashed="yes" rot="R90">
 <attribute name="NAME" x="24.70600625" y="15.117321875" size="0.6096" layer="25" rot="R180"/>
 </element>
-<element name="U3" library="drivers" package="SOT89-5-A" value="PT4115B89E-A2" x="23.97204375" y="8.120265625" smashed="yes" rot="R90">
+<element name="U3" library="drivers" package="SOT89-5" value="PT4115B89E" x="23.97204375" y="8.120265625" smashed="yes" rot="R90">
 <attribute name="NAME" x="24.67054375" y="6.596265625" size="0.6096" layer="25" rot="R180"/>
 </element>
@@
 <attribute name="VALUE" x="32.385" y="34.036" size="0.0254" layer="27"/>
 </element>
-<element name="TP3" library="testpad" package="B1,27" value="PTR1B1,27" x="40.64" y="19.05" smashed="yes">
-<attribute name="TP_SIGNAL_NAME" value="" x="40.005" y="17.145" size="1" layer="37"/>
-<attribute name="VALUE" x="40.005" y="18.288" size="0.0254" layer="27"/>
-</element>
-<element name="TP4" library="testpad" package="B1,27" value="PTR1B1,27" x="40.513" y="2.159" smashed="yes">
-<attribute name="TP_SIGNAL_NAME" value="" x="39.878" y="0.254" size="1" layer="37"/>
-<attribute name="VALUE" x="39.878" y="1.397" size="0.0254" layer="27"/>
-</element>
-<element name="TP5" library="testpad" package="B1,27" value="PTR1B1,27" x="40.64" y="10.16" smashed="yes">
-<attribute name="TP_SIGNAL_NAME" value="" x="40.005" y="8.255" size="1" layer="37"/>
-<attribute name="VALUE" x="40.005" y="9.398" size="0.0254" layer="27"/>
-</element>
-<element name="TP6" library="testpad" package="B1,27" value="PTR1B1,27" x="38.1" y="19.05" smashed="yes">
-<attribute name="TP_SIGNAL_NAME" value="" x="37.465" y="17.145" size="1" layer="37"/>
-<attribute name="VALUE" x="37.465" y="18.288" size="0.0254" layer="27"/>
-</element>
-<element name="TP7" library="testpad" package="B1,27" value="PTR1B1,27" x="38.1" y="10.16" smashed="yes">
-<attribute name="TP_SIGNAL_NAME" value="" x="37.465" y="8.255" size="1" layer="37"/>
-<attribute name="VALUE" x="37.465" y="9.398" size="0.0254" layer="27"/>
-</element>
-<element name="TP8" library="testpad" package="B1,27" value="PTR1B1,27" x="37.592" y="2.159" smashed="yes">
-<attribute name="TP_SIGNAL_NAME" value="" x="36.957" y="0.254" size="1" layer="37"/>
-<attribute name="VALUE" x="36.957" y="1.397" size="0.0254" layer="27"/>
+<element name="TP3" library="testpad" package="B1,27" value="PTR1B1,27" x="39.37" y="19.05" smashed="yes">
+<attribute name="TP_SIGNAL_NAME" value="" x="38.735" y="17.145" size="1" layer="37"/>
+<attribute name="VALUE" x="38.735" y="18.288" size="0.0254" layer="27"/>
+</element>
+<element name="TP4" library="testpad" package="B1,27" value="PTR1B1,27" x="39.243" y="2.159" smashed="yes">
+<attribute name="TP_SIGNAL_NAME" value="" x="38.608" y="0.254" size="1" layer="37"/>
+<attribute name="VALUE" x="38.608" y="1.397" size="0.0254" layer="27"/>
+</element>
+<element name="TP5" library="testpad" package="B1,27" value="PTR1B1,27" x="39.37" y="10.16" smashed="yes">
+<attribute name="TP_SIGNAL_NAME" value="" x="38.735" y="8.255" size="1" layer="37"/>
+<attribute name="VALUE" x="38.735" y="9.398" size="0.0254" layer="27"/>
+</element>
+<element name="TP6" library="testpad" package="B1,27" value="PTR1B1,27" x="36.83" y="19.05" smashed="yes">
+<attribute name="TP_SIGNAL_NAME" value="" x="36.195" y="17.145" size="1" layer="37"/>
+<attribute name="VALUE" x="36.195" y="18.288" size="0.0254" layer="27"/>
+</element>
+<element name="TP7" library="testpad" package="B1,27" value="PTR1B1,27" x="36.83" y="10.16" smashed="yes">
+<attribute name="TP_SIGNAL_NAME" value="" x="36.195" y="8.255" size="1" layer="37"/>
+<attribute name="VALUE" x="36.195" y="9.398" size="0.0254" layer="27"/>
+</element>
+<element name="TP8" library="testpad" package="B1,27" value="PTR1B1,27" x="36.322" y="2.159" smashed="yes">
+<attribute name="TP_SIGNAL_NAME" value="" x="35.687" y="0.254" size="1" layer="37"/>
+<attribute name="VALUE" x="35.687" y="1.397" size="0.0254" layer="27"/>
 </element>
 </elements>
@@
 <wire x1="28.5125375" y1="26.0995375" x2="27.178" y2="25.908" width="0.6096" layer="1"/>
 <wire x1="27.178" y1="25.908" x2="26.136125" y2="25.938515625" width="0.6096" layer="1"/>
-<wire x1="36.83" y1="24.13" x2="36.83" y2="20.32" width="0.4064" layer="1"/>
-<wire x1="36.83" y1="20.32" x2="38.1" y2="19.05" width="0.4064" layer="1"/>
+<wire x1="36.83" y1="24.13" x2="36.83" y2="19.05" width="0.4064" layer="1"/>
 </signal>
 <signal name="BLUE">
@@
 <wire x1="27.432" y1="10.287" x2="35.687" y2="10.16" width="0.4064" layer="1"/>
 <wire x1="36.83" y1="6.35" x2="36.83" y2="3.81" width="0.4064" layer="1"/>
-<wire x1="36.83" y1="3.81" x2="37.592" y2="2.159" width="0.4064" layer="1"/>
-<wire x1="35.687" y1="10.16" x2="36.83" y2="9.017" width="0.4064" layer="1"/>
-<wire x1="36.83" y1="9.017" x2="36.83" y2="6.35" width="0.4064" layer="1"/>
+<wire x1="36.83" y1="3.81" x2="36.322" y2="2.159" width="0.4064" layer="1"/>
+<wire x1="35.687" y1="10.16" x2="36.83" y2="7.747" width="0.4064" layer="1"/>
+<wire x1="36.83" y1="7.747" x2="36.83" y2="6.35" width="0.4064" layer="1"/>
 </signal>
 <signal name="GREEN">
@@
 <wire x1="36.87621875" y1="17.728784375" x2="36.83" y2="15.24" width="0.6096" layer="1"/>
 <wire x1="36.83" y1="15.24" x2="36.703" y2="12.573" width="0.6096" layer="1"/>
-<wire x1="36.703" y1="12.573" x2="38.1" y2="10.16" width="0.6096" layer="1"/>
+<wire x1="36.703" y1="12.573" x2="36.83" y2="10.16" width="0.6096" layer="1"/>
 </signal>
 <signal name="+12V">
@@
 <wire x1="39.243" y1="26.162" x2="38.1" y2="25.654" width="0.6096" layer="1"/>
 <wire x1="38.1" y1="22.225" x2="38.1" y2="20.574" width="0.6096" layer="1"/>
-<wire x1="38.1" y1="20.574" x2="40.64" y2="19.05" width="0.6096" layer="1"/>
+<wire x1="38.1" y1="20.574" x2="39.37" y2="19.05" width="0.6096" layer="1"/>
 </signal>
 <signal name="N$15">
@@
 <contactref element="TP4" pad="TP"/>
 <wire x1="38.1" y1="4.445" x2="38.735" y2="4.445" width="0.6096" layer="1"/>
-<wire x1="38.735" y1="4.445" x2="40.513" y2="2.159" width="0.6096" layer="1"/>
+<wire x1="38.735" y1="4.445" x2="39.243" y2="2.159" width="0.6096" layer="1"/>
 <wire x1="41.91" y1="4.191" x2="41.91" y2="3.81" width="0.6096" layer="1"/>
-<wire x1="41.91" y1="3.81" x2="40.513" y2="2.159" width="0.6096" layer="1"/>
+<wire x1="41.91" y1="3.81" x2="39.243" y2="2.159" width="0.6096" layer="1"/>
 </signal>
 <signal name="N$18">
@@
 <wire x1="37.338" y1="30.861" x2="35.306" y2="28.829" width="0.6096" layer="16"/>
 <wire x1="38.1" y1="13.335" x2="38.735" y2="11.811" width="0.6096" layer="1"/>
-<wire x1="38.735" y1="11.811" x2="40.64" y2="10.16" width="0.6096" layer="1"/>
+<wire x1="38.735" y1="11.811" x2="39.37" y2="10.16" width="0.6096" layer="1"/>
 <wire x1="41.91" y1="15.621" x2="41.91" y2="13.716" width="0.6096" layer="1"/>
 <wire x1="41.91" y1="13.716" x2="38.1" y2="13.335" width="0.6096" layer="1"/>
