File: PixiFlood_PTH.sch (EAGLE design)
At the start: 37 parts, among them IC1 WS2811-SOP8, IC2 78L05Z, T1 2N3904, T2 2N3904, T3 2N3904, U1 PT4115B89E, U2 PT4115B89E, U3 PT4115B89E, X1 22-23-2031, X2 22-23-2031

Commit message: Version 9 of the Driver
Parts:
- R1, R2, R3: value .33R -> .3R
- U1, U2, U3: value PT4115B89E -> PT4115B89E-A2; device drivers:PT4115B89E -> drivers:PT4115B89E-A2
Other:
- moved on the sheet: R4, R5, R6, TP5
Changed lines of the file:
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@@
 <?xml version="1.0" encoding="utf-8"?>
 <!DOCTYPE eagle SYSTEM "eagle.dtd">
-<eagle version="7.2.0">
+<eagle version="7.3.0">
 <drawing>
 <settings>
@@
 </classes>
 <parts>
-<part name="U1" library="drivers" deviceset="PT4115" device="B89E"/>
-<part name="U2" library="drivers" deviceset="PT4115" device="B89E"/>
-<part name="U3" library="drivers" deviceset="PT4115" device="B89E"/>
+<part name="U1" library="drivers" deviceset="PT4115" device="B89E-A2" value="PT4115B89E-A2"/>
+<part name="U2" library="drivers" deviceset="PT4115" device="B89E-A2" value="PT4115B89E-A2"/>
+<part name="U3" library="drivers" deviceset="PT4115" device="B89E-A2" value="PT4115B89E-A2"/>
 <part name="D1" library="diode" deviceset="DIODE-" device="DO07" value="2N3904"/>
 <part name="D2" library="diode" deviceset="DIODE-" device="DO07" value="2N3904"/>
 <part name="D3" library="diode" deviceset="DIODE-" device="DO07" value="2N3904"/>
-<part name="R1" library="resistor" deviceset="R-US_" device="0204/7" value=".33R"/>
-<part name="R2" library="resistor" deviceset="R-US_" device="0204/7" value=".33R"/>
-<part name="R3" library="resistor" deviceset="R-US_" device="0204/7" value=".33R"/>
+<part name="R1" library="resistor" deviceset="R-US_" device="0204/7" value=".3R"/>
+<part name="R2" library="resistor" deviceset="R-US_" device="0204/7" value=".3R"/>
+<part name="R3" library="resistor" deviceset="R-US_" device="0204/7" value=".3R"/>
 <part name="C1" library="rcl" deviceset="CPOL-US" device="TT2D6L" value="100uF"/>
 <part name="GND4" library="supply1" deviceset="GND" device=""/>
@@
 <attribute name="VALUE" x="-33.02" y="2.54" size="1.778" layer="96"/>
 </instance>
-<instance part="R5" gate="G$1" x="-40.64" y="7.62" smashed="yes" rot="R270">
-<attribute name="NAME" x="-40.8686" y="1.27" size="1.778" layer="95" rot="R90"/>
-<attribute name="VALUE" x="-37.338" y="5.08" size="1.778" layer="96" rot="R90"/>
-</instance>
-<instance part="R6" gate="G$1" x="-45.72" y="7.62" smashed="yes" rot="R270">
-<attribute name="NAME" x="-45.9486" y="1.27" size="1.778" layer="95" rot="R90"/>
-<attribute name="VALUE" x="-42.672" y="5.588" size="1.778" layer="96" rot="R90"/>
-</instance>
-<instance part="R4" gate="G$1" x="-35.56" y="7.62" smashed="yes" rot="R270">
-<attribute name="NAME" x="-35.7886" y="1.27" size="1.778" layer="95" rot="R90"/>
-<attribute name="VALUE" x="-32.258" y="4.826" size="1.778" layer="96" rot="R90"/>
+<instance part="R5" gate="G$1" x="-43.18" y="7.62" smashed="yes" rot="R270">
+<attribute name="NAME" x="-43.4086" y="1.27" size="1.778" layer="95" rot="R90"/>
+<attribute name="VALUE" x="-39.878" y="5.08" size="1.778" layer="96" rot="R90"/>
+</instance>
+<instance part="R6" gate="G$1" x="-48.26" y="7.62" smashed="yes" rot="R270">
+<attribute name="NAME" x="-48.4886" y="1.27" size="1.778" layer="95" rot="R90"/>
+<attribute name="VALUE" x="-45.212" y="5.588" size="1.778" layer="96" rot="R90"/>
+</instance>
+<instance part="R4" gate="G$1" x="-38.1" y="7.62" smashed="yes" rot="R270">
+<attribute name="NAME" x="-38.3286" y="1.27" size="1.778" layer="95" rot="R90"/>
+<attribute name="VALUE" x="-34.798" y="4.826" size="1.778" layer="96" rot="R90"/>
 </instance>
 <instance part="P+2" gate="1" x="-24.13" y="12.7" rot="R270"/>
@@
 <instance part="TP3" gate="G$1" x="-53.34" y="-40.64"/>
 <instance part="TP4" gate="G$1" x="-53.34" y="0" rot="R180"/>
-<instance part="TP5" gate="G$1" x="-45.72" y="-17.78" rot="R180"/>
+<instance part="TP5" gate="G$1" x="-48.26" y="-17.78" rot="R180"/>
 <instance part="TP6" gate="G$1" x="-5.08" y="-35.56"/>
 <instance part="TP7" gate="G$1" x="-5.08" y="-17.78"/>
@@
 <pinref part="P+2" gate="1" pin="+5V"/>
 <pinref part="R5" gate="G$1" pin="1"/>
-<junction x="-40.64" y="12.7"/>
-<wire x1="-45.72" y1="12.7" x2="-40.64" y2="12.7" width="0.1524" layer="91"/>
-<wire x1="-40.64" y1="12.7" x2="-35.56" y2="12.7" width="0.1524" layer="91"/>
+<junction x="-43.18" y="12.7"/>
+<wire x1="-48.26" y1="12.7" x2="-43.18" y2="12.7" width="0.1524" layer="91"/>
+<wire x1="-43.18" y1="12.7" x2="-38.1" y2="12.7" width="0.1524" layer="91"/>
 <pinref part="R4" gate="G$1" pin="1"/>
-<junction x="-35.56" y="12.7"/>
-<wire x1="-35.56" y1="12.7" x2="-26.67" y2="12.7" width="0.1524" layer="91"/>
+<junction x="-38.1" y="12.7"/>
+<wire x1="-38.1" y1="12.7" x2="-26.67" y2="12.7" width="0.1524" layer="91"/>
 <pinref part="R6" gate="G$1" pin="1"/>
 </segment>
@@
 <wire x1="-60.96" y1="-22.86" x2="-53.34" y2="-22.86" width="0.1524" layer="91"/>
 <wire x1="-53.34" y1="-22.86" x2="-53.34" y2="-38.1" width="0.1524" layer="91"/>
-<wire x1="-53.34" y1="-38.1" x2="-35.56" y2="-38.1" width="0.1524" layer="91"/>
+<wire x1="-53.34" y1="-38.1" x2="-38.1" y2="-38.1" width="0.1524" layer="91"/>
 <pinref part="R4" gate="G$1" pin="2"/>
-<wire x1="-35.56" y1="-38.1" x2="-17.78" y2="-38.1" width="0.1524" layer="91"/>
-<wire x1="-35.56" y1="2.54" x2="-35.56" y2="-38.1" width="0.1524" layer="91"/>
-<junction x="-35.56" y="-38.1"/>
+<wire x1="-38.1" y1="-38.1" x2="-17.78" y2="-38.1" width="0.1524" layer="91"/>
+<wire x1="-38.1" y1="2.54" x2="-38.1" y2="-38.1" width="0.1524" layer="91"/>
+<junction x="-38.1" y="-38.1"/>
 <pinref part="TP3" gate="G$1" pin="TP"/>
 <junction x="-53.34" y="-38.1"/>
@@
 <wire x1="-60.96" y1="-17.78" x2="-53.34" y2="-17.78" width="0.1524" layer="91"/>
 <wire x1="-53.34" y1="-17.78" x2="-53.34" y2="-2.54" width="0.1524" layer="91"/>
-<wire x1="-53.34" y1="-2.54" x2="-45.72" y2="-2.54" width="0.1524" layer="91"/>
+<wire x1="-53.34" y1="-2.54" x2="-48.26" y2="-2.54" width="0.1524" layer="91"/>
 <pinref part="R6" gate="G$1" pin="2"/>
-<wire x1="-45.72" y1="-2.54" x2="-35.56" y2="-2.54" width="0.1524" layer="91"/>
-<wire x1="-45.72" y1="2.54" x2="-45.72" y2="-2.54" width="0.1524" layer="91"/>
-<junction x="-45.72" y="-2.54"/>
+<wire x1="-48.26" y1="-2.54" x2="-35.56" y2="-2.54" width="0.1524" layer="91"/>
+<wire x1="-48.26" y1="2.54" x2="-48.26" y2="-2.54" width="0.1524" layer="91"/>
+<junction x="-48.26" y="-2.54"/>
 <pinref part="TP4" gate="G$1" pin="TP"/>
 <junction x="-53.34" y="-2.54"/>
@@
 <pinref part="T2" gate="G1" pin="B"/>
 <pinref part="IC1" gate="G$1" pin="G"/>
-<wire x1="-60.96" y1="-20.32" x2="-45.72" y2="-20.32" width="0.1524" layer="91"/>
+<wire x1="-60.96" y1="-20.32" x2="-48.26" y2="-20.32" width="0.1524" layer="91"/>
 <pinref part="R5" gate="G$1" pin="2"/>
-<wire x1="-45.72" y1="-20.32" x2="-40.64" y2="-20.32" width="0.1524" layer="91"/>
-<wire x1="-40.64" y1="-20.32" x2="-25.4" y2="-20.32" width="0.1524" layer="91"/>
-<wire x1="-40.64" y1="2.54" x2="-40.64" y2="-20.32" width="0.1524" layer="91"/>
-<junction x="-40.64" y="-20.32"/>
+<wire x1="-48.26" y1="-20.32" x2="-43.18" y2="-20.32" width="0.1524" layer="91"/>
+<wire x1="-43.18" y1="-20.32" x2="-25.4" y2="-20.32" width="0.1524" layer="91"/>
+<wire x1="-43.18" y1="2.54" x2="-43.18" y2="-20.32" width="0.1524" layer="91"/>
+<junction x="-43.18" y="-20.32"/>
 <pinref part="TP5" gate="G$1" pin="TP"/>
-<junction x="-45.72" y="-20.32"/>
-</segment>
-</net>
+<junction x="-48.26" y="-20.32"/>
+</segment>
+</net>
