File: PixiFlood_PTH.sch (EAGLE design)
At the start: 37 parts, among them IC1 WS2811-SOP8, IC2 78L05Z, T1 2N3904, T2 2N3904, T3 2N3904, U1 PT4115B89E-A2, U2 PT4115B89E-A2, U3 PT4115B89E-A2, X1 22-23-2031, X2 22-23-2031

Commit message: added 20w board
Parts:
- U1, U2, U3: value PT4115B89E-A2 -> PT4115B89E; device drivers:PT4115B89E-A2 -> drivers:PT4115B89E
Changed lines of the file:
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@@
 </classes>
 <parts>
-<part name="U1" library="drivers" deviceset="PT4115" device="B89E-A2" value="PT4115B89E-A2"/>
-<part name="U2" library="drivers" deviceset="PT4115" device="B89E-A2" value="PT4115B89E-A2"/>
-<part name="U3" library="drivers" deviceset="PT4115" device="B89E-A2" value="PT4115B89E-A2"/>
+<part name="U1" library="drivers" deviceset="PT4115" device="B89E" value="PT4115B89E"/>
+<part name="U2" library="drivers" deviceset="PT4115" device="B89E" value="PT4115B89E"/>
+<part name="U3" library="drivers" deviceset="PT4115" device="B89E" value="PT4115B89E"/>
 <part name="D1" library="diode" deviceset="DIODE-" device="DO07" value="2N3904"/>
 <part name="D2" library="diode" deviceset="DIODE-" device="DO07" value="2N3904"/>
