File: PixiFlood_SMT.brd (EAGLE design)
At the start: 43 x 46 mm, 37 parts, among them IC1 WS2811-SOP8, IC2 78L05Z, T1 2N3904, T2 2N3904, T3 2N3904, U1 PT4115B89E-A2, U2 PT4115B89E-A2, U3 PT4115B89E-A2, X1 22-23-2031, X2 22-23-2031

Commit message: Version 10 of the Driver ********  WORK IN PROGRESS  ***********
Parts:
- T1, T2, T3: value 2N3904 -> BC846; device transistor:TO92 -> transistor:SOT23
- U1, U2, U3: value PT4115B89E-A2 -> PT4115B89E; device drivers:SOT89-5-A -> drivers:SOT89-5
- moved TP5 2.84 mm to (39.4, 12.7)
- moved TP7 2.84 mm to (36.8, 12.7)
- moved TP4 2.01 mm to (39.4, 3.81)
- moved TP8 1.82 mm to (36.8, 3.81)
- moved TP6 1.80 mm to (36.8, 20.3)
- moved TP3 1.63 mm to (39.6, 20.3)
- moved T2 1.27 mm to (38.1, 16.5)
- moved T3 1.27 mm to (38.1, 7.62)
- moved U1 0.57 mm to (24.1, 24.7)
- moved L1 0.52 mm to (31.2, 24.6)
- moved L3 0.52 mm to (31.2, 8.00)
- moved T1 0.52 mm to (38.6, 24.3)
- moved D2 0.46 mm to (23.9, 12.3)
- moved L2 0.28 mm to (31.2, 16.6)
- moved U3 0.25 mm to (24.0, 7.87)
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Connections:
- net BLUE: now also T3.3; no longer T3.1
- net GND: now also T1.2, T2.2, T3.2; no longer T1.3, T2.3, T3.3
- net GREEN: now also T2.3; no longer T2.1
- net N$15: now also T3.1; no longer T3.2
- net N$18: now also T2.1; no longer T2.2
- net N$20: now also T1.1; no longer T1.2
- net RED: now also T1.3; no longer T1.1
Routing:
- net N$1: track 6.57 -> 9.17 mm
- net N$20: track 16.0 -> 13.7 mm
- net N$3: track 60.1 -> 62.3 mm
- net N$18: track 31.4 -> 29.7 mm, vias 1 -> 2
- net RED: track 17.4 -> 19.0 mm
- net N$5: track 7.51 -> 9.14 mm
- net N$9: track 53.5 -> 55.1 mm
- net N$10: track 39.8 -> 40.5 mm
- net BLUE: track 19.0 -> 18.5 mm
- net N$15: track 45.2 -> 45.7 mm, vias 1 -> 2
- net GREEN: track 19.5 -> 19.1 mm, vias 0 -> 2
