File: PixiFlood_SMT.sch (EAGLE design)
At the start: 37 parts, among them IC1 WS2811-SOP8, IC2 78L05Z, T1 2N3904, T2 2N3904, T3 2N3904, U1 PT4115B89E-A2, U2 PT4115B89E-A2, U3 PT4115B89E-A2, X1 22-23-2031, X2 22-23-2031

Commit message: Version 10 of the Driver ********  WORK IN PROGRESS  ***********
Parts:
- T1, T2, T3: value 2N3904 -> BC846; device transistor:2N3904 -> transistor:BC846
- U1, U2, U3: value PT4115B89E-A2 -> PT4115B89E; device drivers:PT4115B89E-A2 -> drivers:PT4115B89E
