File: PixiFlood_20w.sch (EAGLE design)
At the start: 35 parts, among them IC1 WS2811-SOP8, IC3 L78LXXCU/BU, T1 BC846, T2 BC846, T3 BC846, U1 PT4115B89E, U2 PT4115B89E, U3 PT4115B89E, X2 22-23-2041

Commit message: added 20w board
Parts:
- removed IC3: L78LXXCU/BU, regulators:L78LXXCU/BU
- added IC2: 78L05Z, linear:78L05Z
- added X1: 22-23-2031, MyLibrary:22-23-2031
- B1: value LED-BOARDV4 -> LED-BOARD20W-30W; device special:LED-BOARDV4 -> special:LED-BOARD20W-30W
- C2: device rcl:C-USC0805 -> rcl:C-US050-024X044
- D1, D2, D3: device diode:SCHOTTKY-DIODESS16 -> diode:DIODE-DO07
- L1, L2, L3: value SLF7045 -> 82114RPTH_SMD; device inductors:SLF7045 -> inductors:82114RPTH_SMD
- R1, R2, R3: device resistor:R-US_R1206 -> resistor:R-US_0204/7
- R4, R5, R6: device resistor:R-US_R0805 -> resistor:R-US_0204/7
- R7: device rcl:R-US_M0805 -> rcl:R-US_0204/7
- R8, R9: device rcl:R-US_R0805 -> rcl:R-US_0204/7
- T1, T2, T3: value BC846 -> 2N3904; device transistor:BC846 -> transistor:2N3904
- TP1: value PTR1TP20SQ -> PTR1B2,54; device testpad:PTR1TP20SQ -> testpad:PTR1B2,54
- TP2: value PTR1TP20R -> PTR1B2,54; device testpad:PTR1TP20R -> testpad:PTR1B2,54
- X2: value 22-23-2041 -> 22-23-2031; device connectors:22-23-2041 -> MyLibrary:22-23-2031
Connections:
- net +12V: now also IC2.VI, X1.1; no longer IC3.IN
- net +5V: now also IC2.VO; no longer IC3.OUT
- net GND: now also IC2.GND, X1.2; no longer IC3.GND1
- net N$4: now also X1.3; no longer X2.4
Other:
- moved on the sheet: B1BLUE, B1GREEN, B1RED, R7, R9
